Commit message: added the urdf(using the xacro format) for Robotis OP2 in RViz

File: robotis_op_description/urdf/robotis_op2.xacro (robot description, xacro)
@@ -1,8 +1,16 @@
-<?xml version="1.0" ?>
-<robot name="darwinOP">
-<link name="base_link"/>
+<?xml version="1.0"?>
+<!-- set the robot's name -->
+<robot name="robotis_op2" xmlns:xacro="http://www.ros.org/wiki/xacro">
+  <!-- Constants for robot dimensions -->
+  <xacro:property name="PI" value="3.1415926535897931"/>
+  <!-- Import all Gazebo-customization elements, including Gazebo colors -->
+<!--   <xacro:include filename="$(find robotis_op_description)/urdf/robotis_op2.gazebo" /> -->
+  <!-- Import Rviz colors -->
+  <xacro:include filename="$(find robotis_op_description)/urdf/materials.xacro" />
+  <link name="base_link"/>
   <joint name="base_link_to_body" type="fixed">
     <parent link="base_link"/>
     <child link="MP_BODY"/>
+    <origin xyz="0 0 0" rpy="0 0 0"/>
   </joint>
   <link name="MP_BODY">
@@ -17,13 +25,13 @@
       <geometry>
         <!--box size="0.102 0.109 0.106" /-->
-        <mesh filename="package://robotis_darwin_description/meshes/body.STL"  scale="1 1 1"/>
-      </geometry>
-      <material name="Grey">
-        <color rgba="0.60 0.60 0.60 1.0"/>
-      </material>
-    </visual>
-    <collision>
-      <geometry>
-        <mesh filename="package://robotis_darwin_description/meshes/body_coll.stl"  scale="1 1 1"/>
+        <mesh filename="package://robotis_op_description/meshes/body.STL"  scale="1 1 1"/>
+      </geometry>
+      <material name="Grey">
+        <color rgba="0.60 0.60 0.60 1.0"/>
+      </material>
+    </visual>
+    <collision>
+      <geometry>
+        <mesh filename="package://robotis_op_description/meshes/body_coll.stl"  scale="1 1 1"/>
       </geometry>
     </collision>
@@ -39,13 +47,13 @@
       <geometry>
         <!--box size="0.045 0.022 0.0325" /-->
-        <mesh filename="package://robotis_darwin_description/meshes/neck.STL"  scale="1 1 1"/>
-      </geometry>
-      <material name="Grey">
-        <color rgba="0.60 0.60 0.60 1.0"/>
-      </material>
-    </visual>
-    <collision>
-      <geometry>
-        <mesh filename="package://robotis_darwin_description/meshes/neck_coll.stl"  scale="1 1 1"/>
+        <mesh filename="package://robotis_op_description/meshes/neck.STL"  scale="1 1 1"/>
+      </geometry>
+      <material name="Grey">
+        <color rgba="0.60 0.60 0.60 1.0"/>
+      </material>
+    </visual>
+    <collision>
+      <geometry>
+        <mesh filename="package://robotis_op_description/meshes/neck_coll.stl"  scale="1 1 1"/>
       </geometry>
     </collision>
@@ -61,13 +69,13 @@
       <geometry>
         <!-- box size="0.0634 0.061 0.033" /-->
-        <mesh filename="package://robotis_darwin_description/meshes/head.STL"  scale="1 1 1"/>
-      </geometry>
-      <material name="Grey">
-        <color rgba="0.60 0.60 0.60 1.0"/>
-      </material>
-    </visual>
-    <collision>
-      <geometry>
-        <mesh filename="package://robotis_darwin_description/meshes/head_coll.stl"  scale="1 1 1"/>
+        <mesh filename="package://robotis_op_description/meshes/head.STL"  scale="1 1 1"/>
+      </geometry>
+      <material name="Grey">
+        <color rgba="0.60 0.60 0.60 1.0"/>
+      </material>
+    </visual>
+    <collision>
+      <geometry>
+        <mesh filename="package://robotis_op_description/meshes/head_coll.stl"  scale="1 1 1"/>
       </geometry>
     </collision>
@@ -104,13 +112,13 @@
       <geometry>
         <!--box size="0.016 0.033 0.02165" /-->
-        <mesh filename="package://robotis_darwin_description/meshes/shoulder_l.STL"  scale="1 1 1"/>
-      </geometry>
-      <material name="Grey">
-        <color rgba="0.60 0.60 0.60 1.0"/>
-      </material>
-    </visual>
-    <collision>
-      <geometry>
-        <mesh filename="package://robotis_darwin_description/meshes/shoulder_l_coll.stl"  scale="1 1 1"/>
+        <mesh filename="package://robotis_op_description/meshes/shoulder_l.STL"  scale="1 1 1"/>
+      </geometry>
+      <material name="Grey">
+        <color rgba="0.60 0.60 0.60 1.0"/>
+      </material>
+    </visual>
+    <collision>
+      <geometry>
+        <mesh filename="package://robotis_op_description/meshes/shoulder_l_coll.stl"  scale="1 1 1"/>
       </geometry>
     </collision>
@@ -126,13 +134,13 @@
       <geometry>
         <!--box size="0.06 0.032 0.035" /-->
-        <mesh filename="package://robotis_darwin_description/meshes/arm_high_l.STL"  scale="1 1 1"/>
-      </geometry>
-      <material name="Grey">
-        <color rgba="0.60 0.60 0.60 1.0"/>
-      </material>
-    </visual>
-    <collision>
-      <geometry>
-        <mesh filename="package://robotis_darwin_description/meshes/arm_high_l_coll.stl"  scale="1 1 1"/>
+        <mesh filename="package://robotis_op_description/meshes/arm_high_l.STL"  scale="1 1 1"/>
+      </geometry>
+      <material name="Grey">
+        <color rgba="0.60 0.60 0.60 1.0"/>
+      </material>
+    </visual>
+    <collision>
+      <geometry>
+        <mesh filename="package://robotis_op_description/meshes/arm_high_l_coll.stl"  scale="1 1 1"/>
       </geometry>
     </collision>
@@ -271,5 +279,5 @@
       <geometry>
         <!--box size="0.016 0.033 0.02165" /-->
-        <mesh filename="package://robotis_darwin_description/meshes/shoulder_r.STL"  scale="1 1 1"/>
+        <mesh filename="package://robotis_op_description/meshes/shoulder_r.STL"  scale="1 1 1"/>
       </geometry>
       <material name="Grey">
@@ -280,5 +288,5 @@
       <origin xyz="0 0 0" rpy="1.5707963  0 3.14" />
       <geometry>
-        <mesh filename="package://robotis_darwin_description/meshes/shoulder_r_coll.stl"  scale="1 1 1"/>
+        <mesh filename="package://robotis_op_description/meshes/shoulder_r_coll.stl"  scale="1 1 1"/>
       </geometry>
     </collision>
@@ -294,13 +302,13 @@
       <geometry>
         <!--box size="0.06 0.032 0.035"/-->
-        <mesh filename="package://robotis_darwin_description/meshes/arm_high_r.STL"  scale="1 1 1"/>
-      </geometry>
-      <material name="Grey">
-        <color rgba="0.60 0.60 0.60 1.0"/>
-      </material>
-    </visual>
-    <collision>
-      <geometry>
-        <mesh filename="package://robotis_darwin_description/meshes/arm_high_r_coll.stl"  scale="1 1 1"/>
+        <mesh filename="package://robotis_op_description/meshes/arm_high_r.STL"  scale="1 1 1"/>
+      </geometry>
+      <material name="Grey">
+        <color rgba="0.60 0.60 0.60 1.0"/>
+      </material>
+    </visual>
+    <collision>
+      <geometry>
+        <mesh filename="package://robotis_op_description/meshes/arm_high_r_coll.stl"  scale="1 1 1"/>
       </geometry>
     </collision>
@@ -418,13 +426,13 @@
       <geometry>
         <!--box size="0.045 0.08175 0.028652" /-->
-        <mesh filename="package://robotis_darwin_description/meshes/pelvis_l.STL"  scale="1 1 1"/>
-      </geometry>
-      <material name="Grey">
-        <color rgba="0.60 0.60 0.60 1.0"/>
-      </material>
-    </visual>
-    <collision>
-      <geometry>
-        <mesh filename="package://robotis_darwin_description/meshes/pelvis_l_coll.stl"  scale="1 1 1"/>
+        <mesh filename="package://robotis_op_description/meshes/pelvis_l.STL"  scale="1 1 1"/>
+      </geometry>
+      <material name="Grey">
+        <color rgba="0.60 0.60 0.60 1.0"/>
+      </material>
+    </visual>
+    <collision>
+      <geometry>
+        <mesh filename="package://robotis_op_description/meshes/pelvis_l_coll.stl"  scale="1 1 1"/>
       </geometry>
     </collision>
@@ -440,13 +448,13 @@
       <geometry>
         <!--box size="0.001 0.001 0.001"/-->
-        <mesh filename="package://robotis_darwin_description/meshes/thigh1_l.STL"  scale="1 1 1"/>
-      </geometry>
-      <material name="Grey">
-        <color rgba="0.60 0.60 0.60 1.0"/>
-      </material>
-    </visual>
-    <collision>
-      <geometry>
-        <mesh filename="package://robotis_darwin_description/meshes/thigh1_l_coll.stl"  scale="1 1 1"/>
+        <mesh filename="package://robotis_op_description/meshes/thigh1_l.STL"  scale="1 1 1"/>
+      </geometry>
+      <material name="Grey">
+        <color rgba="0.60 0.60 0.60 1.0"/>
+      </material>
+    </visual>
+    <collision>
+      <geometry>
+        <mesh filename="package://robotis_op_description/meshes/thigh1_l_coll.stl"  scale="1 1 1"/>
       </geometry>
     </collision>
@@ -462,13 +470,13 @@
       <geometry>
         <!--box size="0.093 0.035 0.045"-->
-        <mesh filename="package://robotis_darwin_description/meshes/thigh2_l.STL"  scale="1 1 1"/>
-      </geometry>
-      <material name="Grey">
-        <color rgba="0.60 0.60 0.60 1.0"/>
-      </material>
-    </visual>
-    <collision>
-      <geometry>
-        <mesh filename="package://robotis_darwin_description/meshes/thigh2_l_coll.stl"  scale="1 1 1"/>
+        <mesh filename="package://robotis_op_description/meshes/thigh2_l.STL"  scale="1 1 1"/>
+      </geometry>
+      <material name="Grey">
+        <color rgba="0.60 0.60 0.60 1.0"/>
+      </material>
+    </visual>
+    <collision>
+      <geometry>
+        <mesh filename="package://robotis_op_description/meshes/thigh2_l_coll.stl"  scale="1 1 1"/>
       </geometry>
     </collision>
@@ -484,13 +492,13 @@
       <geometry>
         <!--box size="0.093 0.035 0.045"/-->
-        <mesh filename="package://robotis_darwin_description/meshes/tibia_l.STL"  scale="1 1 1"/>
-      </geometry>
-      <material name="Grey">
-        <color rgba="0.60 0.60 0.60 1.0"/>
-      </material>
-    </visual>
-    <collision>
-      <geometry>
-        <mesh filename="package://robotis_darwin_description/meshes/tibia_l_coll.stl"  scale="1 1 1"/>
+        <mesh filename="package://robotis_op_description/meshes/tibia_l.STL"  scale="1 1 1"/>
+      </geometry>
+      <material name="Grey">
+        <color rgba="0.60 0.60 0.60 1.0"/>
+      </material>
+    </visual>
+    <collision>
+      <geometry>
+        <mesh filename="package://robotis_op_description/meshes/tibia_l_coll.stl"  scale="1 1 1"/>
       </geometry>
     </collision>
@@ -506,13 +514,13 @@
       <geometry>
         <!--box size="0.028652 0.08175 0.045"/-->
-        <mesh filename="package://robotis_darwin_description/meshes/ankle1_l.STL"  scale="1 1 1"/>
-      </geometry>
-      <material name="Grey">
-        <color rgba="0.60 0.60 0.60 1.0"/>
-      </material>
-    </visual>
-    <collision>
-      <geometry>
-        <mesh filename="package://robotis_darwin_description/meshes/ankle1_l_coll.stl"  scale="1 1 1"/>
+        <mesh filename="package://robotis_op_description/meshes/ankle1_l.STL"  scale="1 1 1"/>
+      </geometry>
+      <material name="Grey">
+        <color rgba="0.60 0.60 0.60 1.0"/>
+      </material>
+    </visual>
+    <collision>
+      <geometry>
+        <mesh filename="package://robotis_op_description/meshes/ankle1_l_coll.stl"  scale="1 1 1"/>
       </geometry>
     </collision>
@@ -528,13 +536,13 @@
       <geometry>
         <!--box size="0.008 0.066 0.104"/-->
-        <mesh filename="package://robotis_darwin_description/meshes/ankle2_l.STL"  scale="1 1 1"/>
-      </geometry>
-      <material name="Grey">
-        <color rgba="0.60 0.60 0.60 1.0"/>
-      </material>
-    </visual>
-    <collision>
-      <geometry>
-        <mesh filename="package://robotis_darwin_description/meshes/ankle2_l_coll.stl"  scale="1 1 1"/>
+        <mesh filename="package://robotis_op_description/meshes/ankle2_l.STL"  scale="1 1 1"/>
+      </geometry>
+      <material name="Grey">
+        <color rgba="0.60 0.60 0.60 1.0"/>
+      </material>
+    </visual>
+    <collision>
+      <geometry>
+        <mesh filename="package://robotis_op_description/meshes/ankle2_l_coll.stl"  scale="1 1 1"/>
       </geometry>
     </collision>
@@ -550,13 +558,13 @@
       <geometry>
         <!--box size="0.045 0.08175 0.028652" /-->
-        <mesh filename="package://robotis_darwin_description/meshes/pelvis_r.STL"  scale="1 1 1"/>
-      </geometry>
-      <material name="Grey">
-        <color rgba="0.60 0.60 0.60 1.0"/>
-      </material>
-    </visual>
-    <collision>
-      <geometry>
-        <mesh filename="package://robotis_darwin_description/meshes/pelvis_r_coll.stl"  scale="1 1 1"/>
+        <mesh filename="package://robotis_op_description/meshes/pelvis_r.STL"  scale="1 1 1"/>
+      </geometry>
+      <material name="Grey">
+        <color rgba="0.60 0.60 0.60 1.0"/>
+      </material>
+    </visual>
+    <collision>
+      <geometry>
+        <mesh filename="package://robotis_op_description/meshes/pelvis_r_coll.stl"  scale="1 1 1"/>
       </geometry>
     </collision>
@@ -572,13 +580,13 @@
       <geometry>
         <!--box size="0.001 0.001 0.001"/-->
-        <mesh filename="package://robotis_darwin_description/meshes/thigh1_r.STL"  scale="1 1 1"/>
-      </geometry>
-      <material name="Grey">
-        <color rgba="0.60 0.60 0.60 1.0"/>
-      </material>
-    </visual>
-    <collision>
-      <geometry>
-        <mesh filename="package://robotis_darwin_description/meshes/thigh1_r_coll.stl"  scale="1 1 1"/>
+        <mesh filename="package://robotis_op_description/meshes/thigh1_r.STL"  scale="1 1 1"/>
+      </geometry>
+      <material name="Grey">
+        <color rgba="0.60 0.60 0.60 1.0"/>
+      </material>
+    </visual>
+    <collision>
+      <geometry>
+        <mesh filename="package://robotis_op_description/meshes/thigh1_r_coll.stl"  scale="1 1 1"/>
       </geometry>
     </collision>
@@ -594,13 +602,13 @@
       <geometry>
         <!--box size="0.093 0.035 0.045"/-->
-        <mesh filename="package://robotis_darwin_description/meshes/thigh2_r.STL"  scale="1 1 1"/>
-      </geometry>
-      <material name="Grey">
-        <color rgba="0.60 0.60 0.60 1.0"/>
-      </material>
-    </visual>
-    <collision>
-      <geometry>
-        <mesh filename="package://robotis_darwin_description/meshes/thigh2_r_coll.stl"  scale="1 1 1"/>
+        <mesh filename="package://robotis_op_description/meshes/thigh2_r.STL"  scale="1 1 1"/>
+      </geometry>
+      <material name="Grey">
+        <color rgba="0.60 0.60 0.60 1.0"/>
+      </material>
+    </visual>
+    <collision>
+      <geometry>
+        <mesh filename="package://robotis_op_description/meshes/thigh2_r_coll.stl"  scale="1 1 1"/>
       </geometry>
     </collision>
@@ -616,13 +624,13 @@
       <geometry>
         <!--box size="0.093 0.035 0.045"/-->
-        <mesh filename="package://robotis_darwin_description/meshes/tibia_r.STL"  scale="1 1 1"/>
-      </geometry>
-      <material name="Grey">
-        <color rgba="0.60 0.60 0.60 1.0"/>
-      </material>
-    </visual>
-    <collision>
-      <geometry>
-        <mesh filename="package://robotis_darwin_description/meshes/tibia_r_coll.stl"  scale="1 1 1"/>
+        <mesh filename="package://robotis_op_description/meshes/tibia_r.STL"  scale="1 1 1"/>
+      </geometry>
+      <material name="Grey">
+        <color rgba="0.60 0.60 0.60 1.0"/>
+      </material>
+    </visual>
+    <collision>
+      <geometry>
+        <mesh filename="package://robotis_op_description/meshes/tibia_r_coll.stl"  scale="1 1 1"/>
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