Commit message: cleanup the xacro files

File: robotis_op_description/urdf/materials.xacro (robot description, xacro)
@@ -11,5 +11,5 @@
   </material>
   <material name="grey">
-    <color rgba="0.2 0.2 0.2 1.0"/>
+    <color rgba="0.60 0.60 0.60 1.0"/>
   </material>
   <material name="orange">

File: robotis_op_description/urdf/robotis_op2.xacro (robot description, xacro)
@@ -1,4 +1,4 @@
 <?xml version="1.0"?>
-<!-- set the robot's name -->
+<!-- Set the robot's name -->
 <robot name="robotis_op2" xmlns:xacro="http://www.ros.org/wiki/xacro">
   <!-- Constants for robot dimensions -->
@@ -8,9 +8,10 @@
   <!-- Import Rviz colors -->
   <xacro:include filename="$(find robotis_op_description)/urdf/materials.xacro" />
+  <!--  Set the robot's link and joint -->
   <link name="base_link"/>
   <joint name="base_link_to_body" type="fixed">
     <parent link="base_link"/>
     <child link="MP_BODY"/>
-    <origin xyz="0 0 0" rpy="0 0 0"/>
+    <origin xyz="0 0 0.35" rpy="0 0 0"/>
   </joint>
   <link name="MP_BODY">
@@ -21,13 +22,9 @@
     </inertial>
     <visual>
-      <!--origin xyz="-0.0235 0 -0.03525" rpy="0 0 0" /-->
-      <origin xyz="0 0 0" rpy="0 0 0" />
-      <geometry>
-        <!--box size="0.102 0.109 0.106" /-->
+      <origin xyz="0 0 0" rpy="0 0 0" />
+      <geometry>
         <mesh filename="package://robotis_op_description/meshes/body.STL"  scale="1 1 1"/>
       </geometry>
-      <material name="Grey">
-        <color rgba="0.60 0.60 0.60 1.0"/>
-      </material>
+      <material name="grey"/>
     </visual>
     <collision>
@@ -46,10 +43,7 @@
       <origin xyz="0 0 0" rpy="0 0 0" />
       <geometry>
-        <!--box size="0.045 0.022 0.0325" /-->
         <mesh filename="package://robotis_op_description/meshes/neck.STL"  scale="1 1 1"/>
       </geometry>
-      <material name="Grey">
-        <color rgba="0.60 0.60 0.60 1.0"/>
-      </material>
+      <material name="grey"/>
     </visual>
     <collision>
@@ -68,10 +62,7 @@
       <origin xyz="0 0 0" rpy="0 0 0" />
       <geometry>
-        <!-- box size="0.0634 0.061 0.033" /-->
         <mesh filename="package://robotis_op_description/meshes/head.STL"  scale="1 1 1"/>
       </geometry>
-      <material name="Grey">
-        <color rgba="0.60 0.60 0.60 1.0"/>
-      </material>
+      <material name="grey"/>
     </visual>
     <collision>
@@ -92,7 +83,5 @@
         <box size="0.001 0.001 0.001"  scale="1 1 1"/>
       </geometry>
-      <material name="Grey">
-        <color rgba="0.60 0.60 0.60 1.0"/>
-      </material>
+      <material name="grey"/>
     </visual>
     <collision>
@@ -111,10 +100,7 @@
       <origin xyz="0 0 0" rpy="0 0 0" />
       <geometry>
-        <!--box size="0.016 0.033 0.02165" /-->
         <mesh filename="package://robotis_op_description/meshes/shoulder_l.STL"  scale="1 1 1"/>
       </geometry>
-      <material name="Grey">
-        <color rgba="0.60 0.60 0.60 1.0"/>
-      </material>
+      <material name="grey"/>
     </visual>
     <collision>
@@ -133,10 +119,7 @@
       <origin xyz="0 0 0" rpy="0 0 0" />
       <geometry>
-        <!--box size="0.06 0.032 0.035" /-->
         <mesh filename="package://robotis_op_description/meshes/arm_high_l.STL"  scale="1 1 1"/>
       </geometry>
-      <material name="Grey">
-        <color rgba="0.60 0.60 0.60 1.0"/>
-      </material>
+      <material name="grey"/>
     </visual>
     <collision>
@@ -157,7 +140,5 @@
         <box size="0.032 0.032 0.035" />
       </geometry>
-      <material name="Grey">
-        <color rgba="0.60 0.60 0.60 1.0"/>
-      </material>
+      <material name="grey"/>
     </visual>
     <collision>
@@ -179,7 +160,5 @@
         <box size="0.064 0.032 0.032" />
       </geometry>
-      <material name="Grey">
-        <color rgba="0.60 0.60 0.60 1.0"/>
-      </material>
+      <material name="grey"/>
     </visual>
     <collision>
@@ -201,7 +180,5 @@
         <box size="0.032 0.005 0.032" />
       </geometry>
-      <material name="Grey">
-        <color rgba="0.60 0.60 0.60 1.0"/>
-      </material>
+      <material name="grey"/>
     </visual>
     <collision>
@@ -222,7 +199,5 @@
         <box size="0.032 0.005 0.032" />
       </geometry>
-      <material name="Grey">
-        <color rgba="0.60 0.60 0.60 1.0"/>
-      </material>
+      <material name="grey"/>
     </visual>
     <collision name="COL_MP_ARM_GRIPPER_MOV_L">
@@ -237,7 +212,5 @@
         <box size="0.002 0.01 0.032" />
       </geometry>
-      <material name="Grey">
-        <color rgba="0.60 0.60 0.60 1.0"/>
-      </material>
+      <material name="grey"/>
     </visual>
     <collision name="COL_MP_ARM_GRIPPER_MOV_EXT_L">
@@ -259,7 +232,5 @@
         <box size="0.001 0.001 0.001" />
       </geometry>
-      <material name="Grey">
-        <color rgba="0.60 0.60 0.60 1.0"/>
-      </material>
+      <material name="grey"/>
     </visual>
     <collision>
@@ -278,10 +249,7 @@
       <origin xyz="0 0 0" rpy="0 0 0" />
       <geometry>
-        <!--box size="0.016 0.033 0.02165" /-->
         <mesh filename="package://robotis_op_description/meshes/shoulder_r.STL"  scale="1 1 1"/>
       </geometry>
-      <material name="Grey">
-        <color rgba="0.60 0.60 0.60 1.0"/>
-      </material>
+      <material name="grey"/>
     </visual>
     <collision>
@@ -301,10 +269,7 @@
       <origin xyz="0 0 0" rpy="0 0 0" />
       <geometry>
-        <!--box size="0.06 0.032 0.035"/-->
         <mesh filename="package://robotis_op_description/meshes/arm_high_r.STL"  scale="1 1 1"/>
       </geometry>
-      <material name="Grey">
-        <color rgba="0.60 0.60 0.60 1.0"/>
-      </material>
+      <material name="grey"/>
     </visual>
     <collision>
@@ -325,7 +290,5 @@
         <box size="0.032 0.032 0.035" />
       </geometry>
-      <material name="Grey">
-        <color rgba="0.60 0.60 0.60 1.0"/>
-      </material>
+      <material name="grey"/>
     </visual>
     <collision>
@@ -347,7 +310,5 @@
         <box size="0.064 0.032 0.032" />
       </geometry>
-      <material name="Grey">
-        <color rgba="0.60 0.60 0.60 1.0"/>
-      </material>
+      <material name="grey"/>
     </visual>
     <collision>
@@ -369,7 +330,5 @@
         <box size="0.032 0.005 0.032" />
       </geometry>
-      <material name="Grey">
-        <color rgba="0.60 0.60 0.60 1.0"/>
-      </material>
+      <material name="grey"/>
     </visual>
     <collision>
@@ -390,7 +349,5 @@
         <box size="0.032 0.005 0.032" />
       </geometry>
-      <material name="Grey">
-        <color rgba="0.60 0.60 0.60 1.0"/>
-      </material>
+      <material name="grey"/>
     </visual>
     <collision name="COL_MP_ARM_GRIPPER_MOV_R">
@@ -405,7 +362,5 @@
         <box size="0.002 0.01 0.032" />
       </geometry>
-      <material name="Grey">
-        <color rgba="0.60 0.60 0.60 1.0"/>
-      </material>
+      <material name="grey"/>
     </visual>
     <collision name="COL_MP_ARM_GRIPPER_MOV_EXT_R">
@@ -425,10 +380,7 @@
       <origin xyz="0 0 0" rpy="0 0 0" />
       <geometry>
-        <!--box size="0.045 0.08175 0.028652" /-->
         <mesh filename="package://robotis_op_description/meshes/pelvis_l.STL"  scale="1 1 1"/>
       </geometry>
-      <material name="Grey">
-        <color rgba="0.60 0.60 0.60 1.0"/>
-      </material>
+      <material name="grey"/>
     </visual>
     <collision>
@@ -447,10 +399,7 @@
       <origin xyz="0 0 0" rpy="0 0 0" />
       <geometry>
-        <!--box size="0.001 0.001 0.001"/-->
         <mesh filename="package://robotis_op_description/meshes/thigh1_l.STL"  scale="1 1 1"/>
       </geometry>
-      <material name="Grey">
-        <color rgba="0.60 0.60 0.60 1.0"/>
-      </material>
+      <material name="grey"/>
     </visual>
     <collision>
@@ -469,10 +418,7 @@
       <origin xyz="0 0 0" rpy="0 0 0" />
       <geometry>
-        <!--box size="0.093 0.035 0.045"-->
         <mesh filename="package://robotis_op_description/meshes/thigh2_l.STL"  scale="1 1 1"/>
       </geometry>
-      <material name="Grey">
-        <color rgba="0.60 0.60 0.60 1.0"/>
-      </material>
+      <material name="grey"/>
     </visual>
     <collision>
@@ -491,10 +437,7 @@
       <origin xyz="0 0 0" rpy="0 0 0" />
       <geometry>
-        <!--box size="0.093 0.035 0.045"/-->
         <mesh filename="package://robotis_op_description/meshes/tibia_l.STL"  scale="1 1 1"/>
       </geometry>
-      <material name="Grey">
-        <color rgba="0.60 0.60 0.60 1.0"/>
-      </material>
+      <material name="grey"/>
     </visual>
     <collision>
@@ -513,10 +456,7 @@
       <origin xyz="0 0 0" rpy="0 0 0" />
       <geometry>
-        <!--box size="0.028652 0.08175 0.045"/-->
         <mesh filename="package://robotis_op_description/meshes/ankle1_l.STL"  scale="1 1 1"/>
       </geometry>
-      <material name="Grey">
-        <color rgba="0.60 0.60 0.60 1.0"/>
-      </material>
+      <material name="grey"/>
     </visual>
     <collision>
@@ -535,10 +475,7 @@
       <origin xyz="0 0 0" rpy="0 0 0" />
       <geometry>
-        <!--box size="0.008 0.066 0.104"/-->
         <mesh filename="package://robotis_op_description/meshes/ankle2_l.STL"  scale="1 1 1"/>
       </geometry>
-      <material name="Grey">
-        <color rgba="0.60 0.60 0.60 1.0"/>
-      </material>
+      <material name="grey"/>
     </visual>
     <collision>
@@ -557,10 +494,7 @@
       <origin xyz="0 0 0" rpy="0 0 0" />
       <geometry>
-        <!--box size="0.045 0.08175 0.028652" /-->
         <mesh filename="package://robotis_op_description/meshes/pelvis_r.STL"  scale="1 1 1"/>
       </geometry>
-      <material name="Grey">
-        <color rgba="0.60 0.60 0.60 1.0"/>
-      </material>
+      <material name="grey"/>
     </visual>
     <collision>
@@ -579,10 +513,7 @@
       <origin xyz="0 0 0" rpy="0 0 0" />
       <geometry>
-        <!--box size="0.001 0.001 0.001"/-->
         <mesh filename="package://robotis_op_description/meshes/thigh1_r.STL"  scale="1 1 1"/>
       </geometry>
-      <material name="Grey">
-        <color rgba="0.60 0.60 0.60 1.0"/>
-      </material>
+      <material name="grey"/>
     </visual>
     <collision>
@@ -601,10 +532,7 @@
       <origin xyz="0 0 0" rpy="0 0 0" />
       <geometry>
-        <!--box size="0.093 0.035 0.045"/-->
         <mesh filename="package://robotis_op_description/meshes/thigh2_r.STL"  scale="1 1 1"/>
       </geometry>
-      <material name="Grey">
-        <color rgba="0.60 0.60 0.60 1.0"/>
-      </material>
+      <material name="grey"/>
     </visual>
     <collision>
@@ -623,10 +551,7 @@
       <origin xyz="0 0 0" rpy="0 0 0" />
       <geometry>
-        <!--box size="0.093 0.035 0.045"/-->
         <mesh filename="package://robotis_op_description/meshes/tibia_r.STL"  scale="1 1 1"/>
       </geometry>
-      <material name="Grey">
-        <color rgba="0.60 0.60 0.60 1.0"/>
-      </material>
+      <material name="grey"/>
     </visual>
     <collision>
@@ -645,10 +570,7 @@
       <origin xyz="0 0 0" rpy="0 0 0" />
       <geometry>
-        <!--box size="0.028652 0.08175 0.045"/-->
         <mesh filename="package://robotis_op_description/meshes/ankle1_r.STL"  scale="1 1 1"/>
       </geometry>
-      <material name="Grey">
-        <color rgba="0.60 0.60 0.60 1.0"/>
-      </material>
+      <material name="grey"/>
     </visual>
     <collision>
@@ -667,10 +589,7 @@
       <origin xyz="0 0 0" rpy="0 0 0" />
       <geometry>
-        <!--box size="0.008 0.066 0.104"/-->
         <mesh filename="package://robotis_op_description/meshes/ankle2_r.STL"  scale="1 1 1"/>
       </geometry>
-      <material name="Grey">
-        <color rgba="0.60 0.60 0.60 1.0"/>
-      </material>
+      <material name="grey"/>
     </visual>
     <collision>
@@ -687,7 +606,5 @@
         <box size="0.032 0.005 0.032" />
       </geometry>
-      <material name="Grey">
-        <color rgba="0.60 0.60 0.60 1.0"/>
-      </material>
+      <material name="grey"/>
     </visual>
     -->
