Commit message: added collision mesh macros

File: robotis_op_description/urdf/old/robotis_op2_with_macros.xacro (robot description, xacro)
@@ -25,9 +25,4 @@
       <inertia ixx="3.1081800"  ixy="-0.25460189"  ixz="2.0318174" iyy="6.3787776" iyz="0.16417863" izz="5.3316425" />
     </inertial>
-    <collision>
-      <geometry>
-        <mesh filename="package://robotis_op_description/meshes/body_coll.stl"  scale="1 1 1"/>
-      </geometry>
-    </collision>
   </link>
   <link name="MP_BACK_L">
@@ -37,9 +32,4 @@
       <inertia ixx="3.1081800"  ixy="-0.25460189"  ixz="2.0318174" iyy="6.3787776" iyz="0.16417863" izz="5.3316425" />
     </inertial>
-    <collision>
-      <geometry>
-        <box size="0.001 0.001 0.001"  scale="1 1 1"/>
-      </geometry>
-    </collision>
   </link>
   <link name="MP_SHOULDER_L">
@@ -49,9 +39,4 @@
       <inertia ixx="0.0097758165"  ixy="0.0016911839"  ixz="-0.00045174329" iyx="0.0016911839" iyy="0.010511104" iyz="0.00033406955" izx="-0.00045174329" izy="0.00033406955" izz="0.005476798" />
     </inertial>
-    <collision>
-      <geometry>
-        <mesh filename="package://robotis_op_description/meshes/shoulder_l_coll.stl"  scale="1 1 1"/>
-      </geometry>
-    </collision>
   </link>
   <link name="MP_ARM_HIGH_L" >
@@ -61,9 +46,4 @@
       <inertia ixx="0.12202839"  ixy="-0.0020812626"  ixz="-0.00088143449" iyx="-0.0020812626" iyy="0.038088441" iyz="0.0018251448" izx="-0.00088143449" izy="0.0018251448" izz="0.11340830" />
     </inertial>
-    <collision>
-      <geometry>
-        <mesh filename="package://robotis_op_description/meshes/arm_high_l_coll.stl"  scale="1 1 1"/>
-      </geometry>
-    </collision>
   </link>
   <link name="MP_ARM_LOW_L" >
@@ -73,10 +53,4 @@
       <inertia ixx="0.086855267"  ixy="0.0053020311"  ixz="0.00043636051" iyx="0.0053020311" iyy="0.021192085" iyz="-0.0064855932" izx="0.00043636051" izy="-0.0064855932" izz="0.086845450" />
     </inertial>
-    <collision>
-      <origin xyz="0.016 0.016 0" rpy="0 0 0" />
-      <geometry>
-        <box size="0.032 0.032 0.035" />
-      </geometry>
-    </collision>
   </link>
  <link name="MP_ARM_GRIPPER_FIX_L" >
@@ -86,10 +60,4 @@
       <inertia ixx="0.12202839"  ixy="-0.0020812626"  ixz="-0.00088143449" iyx="-0.0020812626" iyy="0.038088441" iyz="0.0018251448" izx="-0.00088143449" izy="0.0018251448" izz="0.11340830" />
     </inertial>
-    <collision>
-      <origin xyz="0.016 0 0" rpy="0 0 0" />
-      <geometry>
-        <box size="0.064 0.032 0.032" />
-      </geometry>
-    </collision>
   </link>
   <link name="MP_ARM_GRIPPER_FIX_DUMMY_L" >
@@ -99,9 +67,4 @@
       <inertia ixx="0.12202839"  ixy="-0.0020812626"  ixz="-0.00088143449" iyx="-0.0020812626" iyy="0.038088441" iyz="0.0018251448" izx="-0.00088143449" izy="0.0018251448" izz="0.11340830" />
     </inertial>
-    <collision>
-      <geometry>
-        <box size="0.032 0.005 0.032" />
-      </geometry>
-    </collision>
   </link>
   <link name="MP_ARM_GRIPPER_MOV_L" >
@@ -111,16 +74,4 @@
       <inertia ixx="0.12202839"  ixy="-0.0020812626"  ixz="-0.00088143449" iyx="-0.0020812626" iyy="0.038088441" iyz="0.0018251448" izx="-0.00088143449" izy="0.0018251448" izz="0.11340830" />
     </inertial>
-    <collision name="COL_MP_ARM_GRIPPER_MOV_L">
-      <origin xyz="0.016 0 0" rpy="0 0 0" />
-      <geometry>
-        <box size="0.032 0.005 0.032" />
-      </geometry>
-    </collision>
-    <collision name="COL_MP_ARM_GRIPPER_MOV_EXT_L">
-      <origin xyz="0.031 -0.0025 0" rpy="0 0 0" />
-      <geometry>
-        <box size="0.002 0.01 0.032" />
-      </geometry>
-    </collision>
   </link>
   <link name="MP_BACK_R">
@@ -130,9 +81,4 @@
       <inertia ixx="3.1081800"  ixy="-0.25460189"  ixz="2.0318174" iyy="6.3787776" iyz="0.16417863" izz="5.3316425" />
     </inertial>
-    <collision>
-      <geometry>
-        <box size="0.001 0.001 0.001" />
-      </geometry>
-    </collision>
   </link>
   <link name="MP_SHOULDER_R" >
@@ -142,10 +88,4 @@
       <inertia ixx="0.0097758165"  ixy="0.0016911839"  ixz="-0.00045174329" iyx="0.0016911839" iyy="0.010511104" iyz="0.00033406955" izx="-0.00045174329" izy="0.00033406955" izz="0.005476798" />
     </inertial>
-    <collision>
-      <origin xyz="0 0 0" rpy="1.5707963  0 3.14" />
-      <geometry>
-        <mesh filename="package://robotis_op_description/meshes/shoulder_r_coll.stl"  scale="1 1 1"/>
-      </geometry>
-    </collision>
   </link>
   <link name="MP_ARM_HIGH_R" >
@@ -155,9 +95,4 @@
       <inertia ixx="0.12202839"  ixy="-0.0020812626"  ixz="-0.00088143449" iyx="-0.0020812626" iyy="0.038088441" iyz="0.0018251448" izx="-0.00088143449" izy="0.0018251448" izz="0.11340830" />
     </inertial>
-    <collision>
-      <geometry>
-        <mesh filename="package://robotis_op_description/meshes/arm_high_r_coll.stl"  scale="1 1 1"/>
-      </geometry>
-    </collision>
   </link>
   <link name="MP_ARM_LOW_R" >
@@ -167,10 +102,4 @@
       <inertia ixx="0.086855267"  ixy="0.0053020311"  ixz="0.00043636051" iyx="0.0053020311" iyy="0.021192085" iyz="-0.0064855932" izx="0.00043636051" izy="-0.0064855932" izz="0.086845450" />
     </inertial>
-    <collision>
-      <origin xyz="0.016 -0.016 0" rpy="0 0 0" />
-      <geometry>
-        <box size="0.032 0.032 0.035" />
-      </geometry>
-    </collision>
   </link>
   <link name="MP_ARM_GRIPPER_FIX_R" >
@@ -180,10 +109,4 @@
       <inertia ixx="0.12202839"  ixy="-0.0020812626"  ixz="-0.00088143449" iyx="-0.0020812626" iyy="0.038088441" iyz="0.0018251448" izx="-0.00088143449" izy="0.0018251448" izz="0.11340830" />
     </inertial>
-    <collision>
-      <origin xyz="0.016 0 0" rpy="0 0 0" />
-      <geometry>
-        <box size="0.064 0.032 0.032" />
-      </geometry>
-    </collision>
   </link>
   <link name="MP_ARM_GRIPPER_FIX_DUMMY_R" >
@@ -193,9 +116,4 @@
       <inertia ixx="0.12202839"  ixy="-0.0020812626"  ixz="-0.00088143449" iyx="-0.0020812626" iyy="0.038088441" iyz="0.0018251448" izx="-0.00088143449" izy="0.0018251448" izz="0.11340830" />
     </inertial>
-    <collision>
-      <geometry>
-        <box size="0.032 0.005 0.032" />
-      </geometry>
-    </collision>
   </link>
   <link name="MP_ARM_GRIPPER_MOV_R" >
@@ -205,16 +123,4 @@
       <inertia ixx="0.12202839"  ixy="-0.0020812626"  ixz="-0.00088143449" iyx="-0.0020812626" iyy="0.038088441" iyz="0.0018251448" izx="-0.00088143449" izy="0.0018251448" izz="0.11340830" />
     </inertial>
-    <collision name="COL_MP_ARM_GRIPPER_MOV_R">
-      <origin xyz="0.016 0 0" rpy="0 0 0" />
-      <geometry>
-        <box size="0.032 0.005 0.032" />
-      </geometry>
-    </collision>
-    <collision name="COL_MP_ARM_GRIPPER_MOV_EXT_R">
-      <origin xyz="0.031 -0.0025 0" rpy="0 0 0" />
-      <geometry>
-        <box size="0.002 0.01 0.032" />
-      </geometry>
-    </collision>
   </link>
   <link name="MP_PELVIS_L" >
@@ -224,9 +130,4 @@
       <inertia ixx="0.12259691"  ixy="0.00071127469"  ixz="0.00081143913" iyx="0.00071127469" iyy="0.11066637" iyz="-0.0071635476" izx="0.00081143913" izy="-0.0071635476" izz="0.041877668" />
     </inertial>
-    <collision>
-      <geometry>
-        <mesh filename="package://robotis_op_description/meshes/pelvis_l_coll.stl"  scale="1 1 1"/>
-      </geometry>
-    </collision>
   </link>
   <link name="MP_THIGH1_L" >
@@ -236,9 +137,4 @@
       <inertia ixx="0.097950272"  ixy="0.0012119368"  ixz="-0.00021223016" iyx="0.00122119368" iyy="0.032848287" iyz="-0.0019474021" izx="-0.00021223016" izy="-0.0019474021" izz="0.11493509" />
     </inertial>
-    <collision>
-      <geometry>
-        <mesh filename="package://robotis_op_description/meshes/thigh1_l_coll.stl"  scale="1 1 1"/>
-      </geometry>
-    </collision>
   </link>
   <link name="MP_THIGH2_L" >
@@ -248,9 +144,4 @@
       <inertia ixx="0.097950272"  ixy="0.0012119368"  ixz="-0.00021223016" iyx="0.00122119368" iyy="0.032848287" iyz="-0.0019474021" izx="-0.00021223016" izy="-0.0019474021" izz="0.11493509" />
     </inertial>
-    <collision>
-      <geometry>
-        <mesh filename="package://robotis_op_description/meshes/thigh2_l_coll.stl"  scale="1 1 1"/>
-      </geometry>
-    </collision>
   </link>
   <link name="MP_TIBIA_L" >
@@ -260,9 +151,4 @@
       <inertia ixx="0.093369608"  ixy="-0.00093567395"  ixz="-0.00023992085" iyx="-0.00093567395" iyy="0.046295534" iyz="-0.012858493" izx="-0.00023992085" izy="-0.012858493" izz="0.11351516" />
     </inertial>
-    <collision>
-      <geometry>
-        <mesh filename="package://robotis_op_description/meshes/tibia_l_coll.stl"  scale="1 1 1"/>
-      </geometry>
-    </collision>
   </link>
   <link name="MP_ANKLE1_L" >
@@ -272,9 +158,4 @@
       <inertia ixx="0.12079175"  ixy="-0.00079781067"  ixz="-0.00039322246" iyx="-0.00079781067" iyy="0.10885465" iyz="0.0070770117" izx="-0.00039322246" izy="0.0070770117" izz="0.041871103" />
     </inertial>
-    <collision>
-      <geometry>
-        <mesh filename="package://robotis_op_description/meshes/ankle1_l_coll.stl"  scale="1 1 1"/>
-      </geometry>
-    </collision>
   </link>
   <link name="MP_ANKLE2_L" >
@@ -284,9 +165,4 @@
       <inertia ixx="0.12079175"  ixy="-0.00079781067"  ixz="-0.00039322246" iyx="-0.00079781067" iyy="0.10885465" iyz="0.0070770117" izx="-0.00039322246" izy="0.0070770117" izz="0.041871103" />
     </inertial>
-    <collision>
-      <geometry>
-        <mesh filename="package://robotis_op_description/meshes/ankle2_l_coll.stl"  scale="1 1 1"/>
-      </geometry>
-    </collision>
   </link>
   <link name="MP_PELVIS_R" >
@@ -296,9 +172,4 @@
       <inertia ixx="0.12259691"  ixy="0.00071127469"  ixz="0.00081143913" iyx="0.00071127469" iyy="0.11066637" iyz="-0.0071635476" izx="0.00081143913" izy="-0.0071635476" izz="0.041877668" />
     </inertial>
-    <collision>
-      <geometry>
-        <mesh filename="package://robotis_op_description/meshes/pelvis_r_coll.stl"  scale="1 1 1"/>
-      </geometry>
-    </collision>
   </link>
   <link name="MP_THIGH1_R" >
@@ -308,9 +179,4 @@
       <inertia ixx="0.097950272"  ixy="0.0012119368"  ixz="-0.00021223016" iyx="0.00122119368" iyy="0.032848287" iyz="-0.0019474021" izx="-0.00021223016" izy="-0.0019474021" izz="0.11493509" />
     </inertial>
-    <collision>
-      <geometry>
-        <mesh filename="package://robotis_op_description/meshes/thigh1_r_coll.stl"  scale="1 1 1"/>
-      </geometry>
-    </collision>
   </link>
   <link name="MP_THIGH2_R" >
@@ -320,9 +186,4 @@
       <inertia ixx="0.097950272"  ixy="0.0012119368"  ixz="-0.00021223016" iyx="0.00122119368" iyy="0.032848287" iyz="-0.0019474021" izx="-0.00021223016" izy="-0.0019474021" izz="0.11493509" />
     </inertial>
-    <collision>
-      <geometry>
-        <mesh filename="package://robotis_op_description/meshes/thigh2_r_coll.stl"  scale="1 1 1"/>
-      </geometry>
-    </collision>
   </link>
   <link name="MP_TIBIA_R" >
@@ -332,9 +193,4 @@
       <inertia ixx="0.093369608"  ixy="-0.00093567395"  ixz="-0.00023992085" iyx="-0.00093567395" iyy="0.046295534" iyz="-0.012858493" izx="-0.00023992085" izy="-0.012858493" izz="0.11351516" />
     </inertial>
-    <collision>
-      <geometry>
-        <mesh filename="package://robotis_op_description/meshes/tibia_r_coll.stl"  scale="1 1 1"/>
-      </geometry>
-    </collision>
   </link>
   <link name="MP_ANKLE1_R" >
@@ -344,9 +200,4 @@
       <inertia ixx="0.12079175"  ixy="-0.00079781067"  ixz="-0.00039322246" iyx="-0.00079781067" iyy="0.10885465" iyz="0.0070770117" izx="-0.00039322246" izy="0.0070770117" izz="0.041871103" />
     </inertial>
-    <collision>
-      <geometry>
-        <mesh filename="package://robotis_op_description/meshes/ankle1_r_coll.stl"  scale="1 1 1"/>
-      </geometry>
-    </collision>
   </link>
   <link name="MP_ANKLE2_R" >
@@ -356,9 +207,4 @@
       <inertia ixx="0.12079175"  ixy="-0.00079781067"  ixz="-0.00039322246" iyx="-0.00079781067" iyy="0.10885465" iyz="0.0070770117" izx="-0.00039322246" izy="0.0070770117" izz="0.041871103" />
     </inertial>
-    <collision>
-      <geometry>
-        <mesh filename="package://robotis_op_description/meshes/ankle2_r_coll.stl"  scale="1 1 1"/>
-      </geometry>
-    </collision>
   </link>
   <joint name="j_back_l" type="fixed">
